Commit message: version1.0

File: src/environment/src/ugv_forward_obstacle_continuous/urdf/diff_wheeled_robot.xacro (robot description, xacro)
@@ -80,5 +80,5 @@
             <material name="Black" />
         </visual>
-        <collision>
+        <collision name="yyf">
             <origin xyz="0 0 0" rpy="0 0 0 " />
             <geometry>
@@ -90,4 +90,16 @@
         <material>Gazebo/Darkgray</material>
         <turnGravityOff>false</turnGravityOff>
+        <sensor name="contacts" type="contact">
+            <contact>
+                <collision>base_footprint_fixed_joint_lump__yyf_collision</collision>
+            </contact>
+            <plugin name="gazebo_ros_bumper_controller" filename="libgazebo_ros_bumper.so">
+                <alwaysOn>true</alwaysOn>
+                <updateRate>10</updateRate>
+                <frameName>base_link</frameName>
+                <topicName>/robot_bumper</topicName>
+                <visualize>true</visualize>
+            </plugin>
+        </sensor>
     </gazebo>
     <!--Caster front  -->
@@ -235,5 +247,5 @@
             <broadcastTF>1</broadcastTF>
             <wheelTorque>30</wheelTorque>
-            <wheelAcceleration>1.8</wheelAcceleration>
+            <wheelAcceleration>30</wheelAcceleration>
             <commandTopic>cmd_vel</commandTopic>
             <odometryFrame>odom</odometryFrame>
